File: icm20948-breakout.kicad_sch (KiCad schematic)
At the start: 0 parts

Commit message: First cut of schematic
Parts:
- added C4, C5: 100n, symbol Device:C
- added J1: Conn_01x04, symbol Connector_Generic:Conn_01x04
- added R5: 10k, symbol Device:R
- added U1: ICM-20948, Sensor_Motion:InvenSense_QFN-24_3x3mm_P0.4mm, symbol Sensor_Motion:ICM-20948
Connections:
- new net: R5.2, U1.22 (~{CS})
- new net: C4.1, U1.10 (REGOUT)
- new net +1V8: C5.1, R5.1, U1.13 (VDD), U1.8 (VDDIO)
- new net +3.3V: J1.1 (Pin_1)
- new net GND: C4.2, C5.2, J1.2 (Pin_2), U1.18 (GND), U1.20 (GND)
- new net leveltrans/SCL: U1.23 (SCL/SCLK)
- new net leveltrans/SCL1_8: J1.3 (Pin_3)
- new net leveltrans/SDA: U1.24 (SDA/SDI)
- new net leveltrans/SDA1_8: J1.4 (Pin_4)
Other:
- added sheet leveltrans (leveltrans.kicad_sch)
- added sheet psu (psu.kicad_sch)

Commit message: 1.0a
Parts:
- added C6: 100n, Capacitor_SMD:C_0402_1005Metric_Pad0.74x0.62mm_HandSolder, symbol Device:C
- added H1: MountingHole, local:MountingHole_2.2mm_M2, symbol Mechanical:MountingHole
- C4, C5: footprint (none) -> Capacitor_SMD:C_0402_1005Metric_Pad0.74x0.62mm_HandSolder
- J1: footprint (none) -> Connector_PinHeader_2.54mm:PinHeader_1x04_P2.54mm_Vertical
- R5: footprint (none) -> Resistor_SMD:R_0402_1005Metric_Pad0.72x0.64mm_HandSolder
- U1: footprint Sensor_Motion:InvenSense_QFN-24_3x3mm_P0.4mm -> local:InvenSense_QFN-24_3x3mm_P0.4mm
Connections:
- net leveltrans/SCL1_8 is gone; now on net leveltrans/SCL: J1.3 (Pin_3)
- net leveltrans/SDA1_8 is gone; now on net leveltrans/SDA: J1.4 (Pin_4)
- net +1V8: now also C6.1
- net GND: now also C6.2
- net leveltrans/SCL: no longer U1.23 (SCL/SCLK)
- net leveltrans/SDA: no longer U1.24 (SDA/SDI)
- net CS: now reaches R5.2, U1.22 (~{CS})
- net REGOUT: now reaches C4.1, U1.10 (REGOUT)
- net +3.3V renamed +3V3
- new net SCL1_8: U1.23 (SCL/SCLK)
- new net SDA1_8: U1.24 (SDA/SDI)
- no-connect marks 0 -> 5
Other:
- note added: "NB: Xover"
- moved on the sheet: C4, C5, R5

Commit message: A whole bunch of changes after speaking with Jon.
Parts:
- C4, C5, C6: LCSC (none) -> C1525
- J1: footprint Connector_PinHeader_2.54mm:PinHeader_1x04_P2.54mm_Vertical -> local:PinHeader_1x04_P2.54mm_Vertical
- R5: LCSC (none) -> C25744
- U2: renamed from U1; LCSC (none) -> C726001
Changed lines of the file:
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@@
 			)
 		)
-		(property "LCSC" ""
+		(property "LCSC" "C25744	"
 			(at 166.37 86.36 0)
 			(effects
@@
 		(on_board yes)
 		(dnp no)
-		(property "Reference" "U1"
+		(property "Reference" "U2"
 			(at 197.358 114.808 0)
 			(effects
@@
 			)
 		)
-		(property "LCSC" ""
+		(property "LCSC" "C726001"
 			(at 189.23 97.79 0)
 			(effects
@@
 			(project "icm20948-breakout"
 				(path "/f8b90807-004a-4781-bf54-49eb85b4b2a1"
-					(reference "U1")
+					(reference "U2")
 					(unit 1)
 				)
@@
 			)
 		)
-		(property "Footprint" "Connector_PinHeader_2.54mm:PinHeader_1x04_P2.54mm_Vertical"
+		(property "Footprint" "local:PinHeader_1x04_P2.54mm_Vertical"
 			(at 115.57 90.17 0)
 			(effects
@@
 			)
 		)
-		(property "LCSC" ""
+		(property "LCSC" "C1525"
 			(at 210.82 107.95 0)
 			(effects
@@
 			)
 		)
-		(property "LCSC" ""
+		(property "LCSC" "C1525"
 			(at 198.12 69.85 0)
 			(effects
@@
 			)
 		)
-		(property "LCSC" ""
+		(property "LCSC" "C1525"
 			(at 181.61 69.85 0)
 			(effects
