File: icm20948-breakout.kicad_pcb (KiCad board)
At the start: 0 parts

Commit message: Rewrite using KiCad 8
Other:
- copper layers 0 -> 2
Changed lines of the file:
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@@
-(kicad_pcb (version 20221018) (generator pcbnew)
+(kicad_pcb
+	(version 20231231)
+	(generator "pcbnew")
+	(generator_version "7.99")
+	(general
+		(thickness 1.6)
+		(legacy_teardrops no)
+	)
+	(paper "A4")
+	(layers
+		(0 "F.Cu" signal)
+		(31 "B.Cu" signal)
+		(32 "B.Adhes" user "B.Adhesive")
+		(33 "F.Adhes" user "F.Adhesive")
+		(34 "B.Paste" user)
+		(35 "F.Paste" user)
+		(36 "B.SilkS" user "B.Silkscreen")
+		(37 "F.SilkS" user "F.Silkscreen")
+		(38 "B.Mask" user)
+		(39 "F.Mask" user)
+		(40 "Dwgs.User" user "User.Drawings")
+		(41 "Cmts.User" user "User.Comments")
+		(42 "Eco1.User" user "User.Eco1")
+		(43 "Eco2.User" user "User.Eco2")
+		(44 "Edge.Cuts" user)
+		(45 "Margin" user)
+		(46 "B.CrtYd" user "B.Courtyard")
+		(47 "F.CrtYd" user "F.Courtyard")
+		(48 "B.Fab" user)
+		(49 "F.Fab" user)
+		(50 "User.1" user)
+		(51 "User.2" user)
+		(52 "User.3" user)
+		(53 "User.4" user)
+		(54 "User.5" user)
+		(55 "User.6" user)
+		(56 "User.7" user)
+		(57 "User.8" user)
+		(58 "User.9" user)
+	)
+	(setup
+		(pad_to_mask_clearance 0)
+		(allow_soldermask_bridges_in_footprints no)
+		(pcbplotparams
+			(layerselection 0x00010fc_ffffffff)
+			(plot_on_all_layers_selection 0x0000000_00000000)
+			(disableapertmacros no)
+			(usegerberextensions no)
+			(usegerberattributes yes)
+			(usegerberadvancedattributes yes)
+			(creategerberjobfile yes)
+			(dashed_line_dash_ratio 12.000000)
+			(dashed_line_gap_ratio 3.000000)
+			(svgprecision 4)
+			(plotframeref no)
+			(viasonmask no)
+			(mode 1)
+			(useauxorigin no)
+			(hpglpennumber 1)
+			(hpglpenspeed 20)
+			(hpglpendiameter 15.000000)
+			(pdf_front_fp_property_popups yes)
+			(pdf_back_fp_property_popups yes)
+			(dxfpolygonmode yes)
+			(dxfimperialunits yes)
+			(dxfusepcbnewfont yes)
+			(psnegative no)
+			(psa4output no)
+			(plotreference yes)
+			(plotvalue yes)
+			(plotfptext yes)
+			(plotinvisibletext no)
+			(sketchpadsonfab no)
+			(subtractmaskfromsilk no)
+			(outputformat 1)
+			(mirror no)
+			(drillshape 1)
+			(scaleselection 1)
+			(outputdirectory "")
+		)
+	)
+	(net 0 "")
 )

Commit message: 1.0a
Parts:
- added C1: 1u, Capacitor_SMD:C_0603_1608Metric_Pad1.08x0.95mm_HandSolder, F.Cu at (149.9, 95.8)
- added C2: 100n, Capacitor_SMD:C_0603_1608Metric_Pad1.08x0.95mm_HandSolder, F.Cu at (153.8, 98.9)
- added C3: 1u, Capacitor_SMD:C_0603_1608Metric_Pad1.08x0.95mm_HandSolder, F.Cu at (153.8, 100.5)
- added C4: 100n, Capacitor_SMD:C_0402_1005Metric_Pad0.74x0.62mm_HandSolder, F.Cu at (152.6, 102.8)
- added C5: 100n, Capacitor_SMD:C_0402_1005Metric_Pad0.74x0.62mm_HandSolder, F.Cu at (147.1, 102.7)
- added C6: 100n, Capacitor_SMD:C_0402_1005Metric_Pad0.74x0.62mm_HandSolder, F.Cu at (152.6, 105.2)
- added H1: MountingHole, local:MountingHole_2.2mm_M2, F.Cu at (149.9, 108.1)
- added J1: Conn_01x04, Connector_PinHeader_2.54mm:PinHeader_1x04_P2.54mm_Vertical, F.Cu at (153.7, 91.8)
- added Q1: BSS138, Package_TO_SOT_SMD:SOT-23, F.Cu at (150.1, 99.6)
- added Q2: BSS138, Package_TO_SOT_SMD:SOT-23, F.Cu at (146.2, 99.6)
- added R5: 10k, Resistor_SMD:R_0402_1005Metric_Pad0.72x0.64mm_HandSolder, F.Cu at (147.1, 105.2)
- added RN1: 10k, Resistor_SMD:R_Array_Convex_4x0603, F.Cu at (146.4, 95.8)
- added U1: ICM-20948, local:InvenSense_QFN-24_3x3mm_P0.4mm, F.Cu at (149.9, 103.8)
- added U2: MIC5317-1.8xM5, Package_TO_SOT_SMD:SOT-23-5, F.Cu at (153.8, 95.8)
Routing:
- net +1V8: track 0.00 -> 31.9 mm
- net +3V3: track 0.00 -> 23.7 mm
- net GND: track 0.00 -> 21.5 mm, vias 0 -> 10
- net /SCL1_8: track 0.00 -> 17.9 mm
- net /SDA1_8: track 0.00 -> 14.0 mm
- net /leveltrans/SCL: track 0.00 -> 9.66 mm
- net /leveltrans/SDA: track 0.00 -> 8.19 mm
- net /CS: track 0.00 -> 1.59 mm
- net /REGOUT: track 0.00 -> 1.31 mm
- added copper zone on B.Cu, net GND
Other:
- board outline added: 11.6 x 20.8 mm
- board text added: "3V3 GND SCL SDA"
- board text added: "ICM20948 breakout"
- board text added: "JLCJLCJLCJLC"
- board text added: "mjd@afork.com"
- board text added: "v1.0a 3-Jan-2024"

Commit message: A whole bunch of changes after speaking with Jon.
Parts:
- C2: value 100n -> 10n; footprint Capacitor_SMD:C_0603_1608Metric_Pad1.08x0.95mm_HandSolder -> Capacitor_SMD:C_0402_1005Metric_Pad0.74x0.62mm_HandSolder
- J1: footprint Connector_PinHeader_2.54mm:PinHeader_1x04_P2.54mm_Vertical -> local:PinHeader_1x04_P2.54mm_Vertical
- Q1, Q2: value BSS138 -> RJU003N03; footprint Package_TO_SOT_SMD:SOT-23 -> Package_TO_SOT_SMD:SOT-323_SC-70_Handsoldering
- U1: renamed from U2; value MIC5317-1.8xM5 -> RS3221-1.8
- moved C5 4.23 mm to (150.4, 100.1), turned to 180 degrees
- moved R5 3.39 mm to (146.8, 101.8), turned to -90 degrees
- moved Q1 3.11 mm to (149.7, 96.5)
- moved C1 1.70 mm to (150.3, 94.2), turned to 180 degrees
- moved Q2 1.15 mm to (146.5, 98.5)
- moved C6 1.11 mm to (152.6, 104.1)
- moved U2 1.11 mm to (149.9, 102.6)
- moved H1 1.11 mm to (149.9, 107.0)
- moved C3 1.05 mm to (153.9, 99.5)
- moved C2 0.97 mm to (153.4, 98.0), turned to 0 degrees
- moved C4 0.95 mm to (152.6, 101.8)
- moved RN1 0.90 mm to (145.7, 95.3)
- moved U1 0.30 mm to (153.8, 95.5)
- renumbered U1 to U2
Connections:
- C2 pad 1: +1V8 -> /psu/BP
- U1 pad 4: unconnected-(U2-NC-Pad4) (its old number) -> /psu/BP
Routing:
- net +1V8: track 31.9 -> 26.9 mm
- net GND: track 21.5 -> 17.5 mm, vias 10 -> 9
- net /SDA1_8: track 14.0 -> 10.2 mm
- net +3V3: track 23.7 -> 21.0 mm
- net /SCL1_8: track 17.9 -> 15.5 mm
- net /leveltrans/SCL: track 9.66 -> 8.15 mm
- net /psu/BP: track 0.00 -> 1.42 mm
- net /REGOUT: track 1.31 -> 1.93 mm
- added copper zone on F.Cu, net +1V8
Other:
- board size 11.6 x 20.8 mm -> 11.6 x 19.6 mm
- board text added: "v1.1a 6-Jan-2024"
- board text removed: "v1.0a 3-Jan-2024"

Commit message: Changes for v1.1b
Parts:
- C1, C3: footprint Capacitor_SMD:C_0603_1608Metric_Pad1.08x0.95mm_HandSolder -> Capacitor_SMD:C_0402_1005Metric_Pad0.74x0.62mm_HandSolder
- Q1, Q2: footprint Package_TO_SOT_SMD:SOT-323_SC-70_Handsoldering -> local:SOT-323_SC-70_Handsoldering
- moved C2 4.63 mm to (151.3, 93.9)
- moved C1 3.56 mm to (153.8, 93.9)
- moved R5 3.42 mm to (148.4, 98.8), turned to 180 degrees
- moved U1 1.43 mm to (152.6, 96.1), turned to 180 degrees
- moved C4 1.40 mm to (152.6, 100.5)
- moved C6 1.37 mm to (152.6, 102.7)
- moved Q1 1.30 mm to (148.6, 95.8), turned to -90 degrees
- moved Q2 1.27 mm to (145.9, 99.6), turned to -90 degrees
- moved C5 1.05 mm to (150.8, 99.2)
- moved H1 0.94 mm to (149.9, 106.0)
- moved U2 0.94 mm to (149.9, 101.7)
- moved C3 0.91 mm to (153.6, 98.7), turned to 0 degrees
Routing:
- net GND: track 17.5 -> 30.8 mm, vias 9 -> 7
- net /leveltrans/SCL: track 8.15 -> 4.75 mm
- net +1V8: track 26.9 -> 24.1 mm
- net /CS: track 1.76 -> 4.10 mm
- net /SCL1_8: track 15.5 -> 14.1 mm
- net /SDA1_8: track 10.2 -> 9.18 mm
- net /leveltrans/SDA: track 8.30 -> 7.56 mm
- net /REGOUT: track 1.93 -> 1.42 mm
Other:
- board size 11.6 x 19.6 mm -> 11.6 x 18.5 mm
- board text added: "v1.1b 6-Jan-2024"
- board text removed: "v1.1a 6-Jan-2024"
