File: leveltrans.kicad_sch (KiCad schematic)
At the start: 6 parts, among them Q1 BSS138, Q2 BSS138

Commit message: 1.0a
Parts:
- removed R1, R2, R3, R4: R, symbol Device:R
- added RN1: 10k, Resistor_SMD:R_Array_Convex_4x0603, symbol Device:R_Pack04_Split
Connections:
- net +1V8: now also RN1.1 (R1.1), RN1.2 (R2.1)
- net SCL: now also RN1.3 (R3.1)
- net SCL1_8: now also RN1.7 (R2.2)
- net SDA: now also RN1.4 (R4.1)
- net SDA1_8: now also RN1.8 (R1.2)
- new net +3V3: RN1.5 (R4.2), RN1.6 (R3.2)

Commit message: A whole bunch of changes after speaking with Jon.
Parts:
- Q1, Q2: value BSS138 -> RJU003N03; footprint Package_TO_SOT_SMD:SOT-23 -> Package_TO_SOT_SMD:SOT-323_SC-70_Handsoldering; LCSC (none) -> C308741
Changed lines of the file:
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@@
 			)
 		)
-		(property "Value" "BSS138"
+		(property "Value" "RJU003N03 "
 			(at 137.16 92.4094 90)
 			(effects
@@
 			)
 		)
-		(property "Footprint" "Package_TO_SOT_SMD:SOT-23"
+		(property "Footprint" "Package_TO_SOT_SMD:SOT-323_SC-70_Handsoldering"
 			(at 135.255 88.9 0)
 			(effects
@@
 			)
 		)
-		(property "Datasheet" "https://www.onsemi.com/pub/Collateral/BSS138-D.PDF"
+		(property "Datasheet" "https://datasheet.lcsc.com/lcsc/1811131653_ROHM-Semicon-RJU003N03T106_C308741.pdf"
 			(at 133.35 88.9 0)
 			(effects
@@
 			)
 		)
-		(property "LCSC" ""
+		(property "LCSC" "C308741"
 			(at 137.16 83.82 0)
 			(effects
@@
 			)
 		)
-		(property "Value" "BSS138"
+		(property "Value" "RJU003N03 "
 			(at 128.27 102.5694 90)
 			(effects
@@
 			)
 		)
-		(property "Footprint" "Package_TO_SOT_SMD:SOT-23"
+		(property "Footprint" "Package_TO_SOT_SMD:SOT-323_SC-70_Handsoldering"
 			(at 126.365 99.06 0)
 			(effects
@@
 			)
 		)
-		(property "Datasheet" "https://www.onsemi.com/pub/Collateral/BSS138-D.PDF"
+		(property "Datasheet" "https://datasheet.lcsc.com/lcsc/1811131653_ROHM-Semicon-RJU003N03T106_C308741.pdf"
 			(at 124.46 99.06 0)
 			(effects
@@
 			)
 		)
-		(property "LCSC" ""
+		(property "LCSC" "C308741"
 			(at 128.27 93.98 0)
 			(effects

Commit message: Changes for v1.1b
Parts:
- Q1, Q2: footprint Package_TO_SOT_SMD:SOT-323_SC-70_Handsoldering -> local:SOT-323_SC-70_Handsoldering
Changed lines of the file:
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@@
 			)
 		)
-		(property "Footprint" "Package_TO_SOT_SMD:SOT-323_SC-70_Handsoldering"
+		(property "Footprint" "local:SOT-323_SC-70_Handsoldering"
 			(at 135.255 88.9 0)
 			(effects
@@
 			)
 		)
-		(property "Footprint" "Package_TO_SOT_SMD:SOT-323_SC-70_Handsoldering"
+		(property "Footprint" "local:SOT-323_SC-70_Handsoldering"
 			(at 126.365 99.06 0)
 			(effects
