File: psu.kicad_sch (KiCad schematic)
At the start: 4 parts, among them U2 MIC5317-1.8xM5

Commit message: 1.0a
Parts:
- C1, C2, C3: footprint (none) -> Capacitor_SMD:C_0603_1608Metric_Pad1.08x0.95mm_HandSolder
Changed lines of the file:
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@@
 	(wire
 		(pts
-			(xy 135.89 63.5) (xy 135.89 66.04)
+			(xy 135.89 62.23) (xy 135.89 66.04)
 		)
 		(stroke
@@
 	(symbol
 		(lib_id "power:PWR_FLAG")
-		(at 135.89 63.5 0)
+		(at 135.89 62.23 0)
 		(unit 1)
 		(exclude_from_sim no)
@@
 		(fields_autoplaced yes)
 		(property "Reference" "#FLG03"
-			(at 135.89 61.595 0)
+			(at 135.89 60.325 0)
 			(effects
 				(font
@@
 		)
 		(property "Value" "PWR_FLAG"
-			(at 135.89 59.3669 0)
+			(at 135.89 58.0969 0)
 			(effects
 				(font
@@
 		)
 		(property "Footprint" ""
-			(at 135.89 63.5 0)
+			(at 135.89 62.23 0)
 			(effects
 				(font
@@
 		)
 		(property "Datasheet" "~"
-			(at 135.89 63.5 0)
+			(at 135.89 62.23 0)
 			(effects
 				(font
@@
 		)
 		(property "Description" "Special symbol for telling ERC where power comes from"
-			(at 135.89 63.5 0)
+			(at 135.89 62.23 0)
 			(effects
 				(font
@@
 			)
 		)
-		(property "Footprint" ""
+		(property "Footprint" "Capacitor_SMD:C_0603_1608Metric_Pad1.08x0.95mm_HandSolder"
 			(at 133.0452 76.2 0)
 			(effects
@@
 			)
 		)
+		(property "LCSC" ""
+			(at 132.08 72.39 0)
+			(effects
+				(font
+					(size 1.27 1.27)
+				)
+				(hide yes)
+			)
+		)
+		(property "Field-1" ""
+			(at 132.08 72.39 0)
+			(effects
+				(font
+					(size 1.27 1.27)
+				)
+				(hide yes)
+			)
+		)
 		(pin "1"
 		)
@@
 			)
 		)
-		(property "Footprint" ""
+		(property "Footprint" "Capacitor_SMD:C_0603_1608Metric_Pad1.08x0.95mm_HandSolder"
 			(at 124.1552 76.2 0)
 			(effects
@@
 			)
 		)
+		(property "LCSC" ""
+			(at 123.19 72.39 0)
+			(effects
+				(font
+					(size 1.27 1.27)
+				)
+				(hide yes)
+			)
+		)
+		(property "Field-1" ""
+			(at 123.19 72.39 0)
+			(effects
+				(font
+					(size 1.27 1.27)
+				)
+				(hide yes)
+			)
+		)
 		(pin "1"
 		)
@@
 			)
 		)
-		(property "Footprint" ""
+		(property "Footprint" "Capacitor_SMD:C_0603_1608Metric_Pad1.08x0.95mm_HandSolder"
 			(at 98.7552 76.2 0)
 			(effects
@@
 			)
 		)
+		(property "LCSC" ""
+			(at 97.79 72.39 0)
+			(effects
+				(font
+					(size 1.27 1.27)
+				)
+				(hide yes)
+			)
+		)
+		(property "Field-1" ""
+			(at 97.79 72.39 0)
+			(effects
+				(font
+					(size 1.27 1.27)
+				)
+				(hide yes)
+			)
+		)
 		(pin "1"
 		)
@@
 			(at 111.76 68.58 0)
 			(effects
+				(font
+					(size 1.27 1.27)
+				)
+				(hide yes)
+			)
+		)
+		(property "LCSC" ""
+			(at 111.76 68.58 0)
+			(effects
+				(font
+					(size 1.27 1.27)
+				)
+				(hide yes)
+			)
+		)
+		(property "Field-1" ""
+			(at 111.76 68.58 0)
+			(effects

Commit message: A whole bunch of changes after speaking with Jon.
Parts:
- C1, C3: LCSC (none) -> C15849
- C2: value 100n -> 10n; footprint Capacitor_SMD:C_0603_1608Metric_Pad1.08x0.95mm_HandSolder -> Capacitor_SMD:C_0402_1005Metric_Pad0.74x0.62mm_HandSolder; LCSC (none) -> C15195
- U1: renamed from U2; value MIC5317-1.8xM5 -> RS3221-1.8; symbol Regulator_Linear:MIC5317-1.8xM5 -> local:RS3221-1.8; LCSC (none) -> C2762317
Connections:
- net +1V8: no longer C2.1
- net BP: now reaches U1.4 (NC)
- net BP: now also C2.1
Changed lines of the file:
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@@
-	)
-	(junction
-		(at 123.19 66.04)
-		(diameter 0)
-		(color 0 0 0 0)
 	)
 	(junction
@@
 	(wire
 		(pts
-			(xy 132.08 66.04) (xy 123.19 66.04)
-		)
-		(stroke
-			(width 0)
-			(type default)
-		)
-	)
-	(wire
-		(pts
-			(xy 123.19 66.04) (xy 119.38 66.04)
+			(xy 119.38 66.04) (xy 132.08 66.04)
 		)
 		(stroke
@@
 	(wire
 		(pts
+			(xy 119.38 68.58) (xy 123.19 68.58)
+		)
+		(stroke
+			(width 0)
+			(type default)
+		)
+	)
+	(wire
+		(pts
 			(xy 97.79 66.04) (xy 101.6 66.04)
 		)
@@
 		(pts
 			(xy 97.79 66.04) (xy 97.79 68.58)
-		)
-		(stroke
-			(width 0)
-			(type default)
-		)
-	)
-	(wire
-		(pts
-			(xy 123.19 68.58) (xy 123.19 66.04)
 		)
 		(stroke
@@
 		)
 	)
+	(label "BP"
+		(at 123.19 68.58 180)
+		(fields_autoplaced yes)
+		(effects
+			(font
+				(size 1.27 1.27)
+			)
+			(justify right bottom)
+		)
+	)
 	(symbol
 		(lib_id "power:GND")
@@
 			)
 		)
-		(property "LCSC" ""
+		(property "LCSC" "C15849"
 			(at 132.08 72.39 0)
 			(effects
@@
 			)
 		)
-		(property "Value" "100n"
+		(property "Value" "10n"
 			(at 126.111 73.6021 0)
 			(effects
@@
 			)
 		)
-		(property "Footprint" "Capacitor_SMD:C_0603_1608Metric_Pad1.08x0.95mm_HandSolder"
+		(property "Footprint" "Capacitor_SMD:C_0402_1005Metric_Pad0.74x0.62mm_HandSolder"
 			(at 124.1552 76.2 0)
 			(effects
@@
 			)
 		)
-		(property "LCSC" ""
+		(property "LCSC" "C15195"
 			(at 123.19 72.39 0)
 			(effects
@@
 			)
 		)
-		(property "LCSC" ""
+		(property "LCSC" "C15849"
 			(at 97.79 72.39 0)
 			(effects
@@
 	)
 	(symbol
-		(lib_id "Regulator_Linear:MIC5317-1.8xM5")
+		(lib_id "local:RS3221-1.8")
 		(at 111.76 68.58 0)
 		(unit 1)
@@
 		(dnp no)
 		(fields_autoplaced yes)
-		(property "Reference" "U2"
+		(property "Reference" "U1"
 			(at 111.76 59.9905 0)
 			(effects
@@
 			)
 		)
-		(property "Value" "MIC5317-1.8xM5"
+		(property "Value" "RS3221-1.8"
 			(at 111.76 62.4148 0)
 			(effects
@@
 		)
 		(property "Footprint" "Package_TO_SOT_SMD:SOT-23-5"
-			(at 111.76 59.69 0)
-			(effects
-				(font
-					(size 1.27 1.27)
-				)
-				(hide yes)
-			)
-		)
-		(property "Datasheet" "https://ww1.microchip.com/downloads/aemDocuments/documents/OTH/ProductDocuments/DataSheets/MIC5317-High-Performance-Single-150mA-LDO-DS20006195B.pdf"
-			(at 104.14 48.26 0)
-			(effects
-				(font
-					(size 1.27 1.27)
-				)
-				(hide yes)
-			)
-		)
-		(property "Description" "150mA Low-dropout Voltage Regulator, Vout 1.8V, Vin up to 6V, SOT23-5"
+			(at 111.76 60.325 0)
+			(effects
+				(font
+					(size 1.27 1.27)
+				)
+				(hide yes)
+			)
+		)
+		(property "Datasheet" "https://datasheet.lcsc.com/lcsc/2304140030_Jiangsu-RUNIC-Tech-RS3221-1-8YF5_C2762317.pdf"
+			(at 111.76 66.04 0)
+			(effects
+				(font
+					(size 1.27 1.27)
+				)
+				(hide yes)
+			)
+		)
+		(property "Description" "200mA low dropout linear regulator, wide input voltage range, 1.8V fixed positive output, SOT-23-5"
 			(at 111.76 68.58 0)
 			(effects
@@
 			)
 		)
-		(property "LCSC" ""
+		(property "LCSC" "C2762317"
 			(at 111.76 68.58 0)
 			(effects
@@
 			)
 		)
-		(property "Field-1" ""
-			(at 111.76 68.58 0)
-			(effects
-				(font
-					(size 1.27 1.27)
-				)
-				(hide yes)
-			)
-		)
 		(pin "2"
 		)
@@
 		(pin "3"
 		)
-		(instances
-			(project "icm20948-breakout"
-				(path "/f8b90807-004a-4781-bf54-49eb85b4b2a1/4e2c07ed-6aea-4860-a988-decce8f290ab"
-					(reference "U2")
-					(unit 1)
-				)
+		(pin "4"
+		)
+		(instances
+			(project "icm20948-breakout"
+				(path "/f8b90807-004a-4781-bf54-49eb85b4b2a1/4e2c07ed-6aea-4860-a988-decce8f290ab"
+					(reference "U1")
+					(unit 1)
+				)

Commit message: Changes for v1.1b
Parts:
- C1, C3: footprint Capacitor_SMD:C_0603_1608Metric_Pad1.08x0.95mm_HandSolder -> Capacitor_SMD:C_0402_1005Metric_Pad0.74x0.62mm_HandSolder; LCSC C15849 -> C52923
Changed lines of the file:
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@@
 			)
 		)
-		(property "Footprint" "Capacitor_SMD:C_0603_1608Metric_Pad1.08x0.95mm_HandSolder"
+		(property "Footprint" "Capacitor_SMD:C_0402_1005Metric_Pad0.74x0.62mm_HandSolder"
 			(at 133.0452 76.2 0)
 			(effects
@@
 			)
 		)
-		(property "LCSC" "C15849"
+		(property "LCSC" "C52923 "
 			(at 132.08 72.39 0)
 			(effects
@@
 			)
 		)
-		(property "Footprint" "Capacitor_SMD:C_0603_1608Metric_Pad1.08x0.95mm_HandSolder"
+		(property "Footprint" "Capacitor_SMD:C_0402_1005Metric_Pad0.74x0.62mm_HandSolder"
 			(at 98.7552 76.2 0)
 			(effects
@@
 			)
 		)
-		(property "LCSC" "C15849"
+		(property "LCSC" "C52923 "
 			(at 97.79 72.39 0)
 			(effects
